File: hdmi-featherwing.kicad_sch (KiCad schematic)
At the start: 0 parts

Commit message: Add HDMI connector to schematic
Parts:
- added J?: HDMI_A, HDMI:HDMI-TH_HYC12-HDMIA19-61, symbol Connector:HDMI_A
- added R? (x8): 270, symbol Device:R
Connections:
- new net: J?.1 (D2+), R?.2
- new net: J?.9 (D0-), R?.2
- new net: J?.3 (D2-), R?.2
- new net: J?.6 (D1-), R?.2
- new net: J?.10 (CK+), R?.2
- new net: J?.7 (D0+), R?.2
- new net: J?.4 (D1+), R?.2
- new net: J?.12 (CK-), R?.2
- new net +5V: J?.18 (+5V)
- new net GND: J?.11 (CKS), J?.17 (GND), J?.2 (D2S), J?.5 (D1S), J?.8 (D0S), J?.SH
- no-connect marks 0 -> 5
